Commit message: refactor ensenso.xacro
add N4x / refactor examples

remove projector- and right_lens-links & projector-objective == sensor-objective

remove objectives / integrate Sx / update stl

update FA *.stl

File: ensenso_description/ensenso.xacro (robot description, xacro)
@@ -7,15 +7,35 @@
   <color rgba="0.0 0.0 0.0 1.0"/>
 </material>
-  <xacro:macro name="ensenso_N_Series" params="camera parent *origin margin">
-    <joint name="${parent}_${camera}_joint" type="fixed">
-      <xacro:insert_block name="origin"/>
-      <parent link="${parent}" />
-      <child link="${camera}_mounting_frame" />
-    </joint>
-    <link name="${camera}_mounting_frame">
+<xacro:macro name="ensenso_Sx_Series" params="name margin:=0.03">
+    <link name="${name}">
       <visual>
         <origin rpy="0 0 0" xyz="0.00 0.0 0.0"/>
         <geometry>
-          <mesh filename="package://ensenso_description/stl_meshes/N30-602-16.stl"/>
+          <mesh filename="package://ensenso_description/stl_meshes/Sx.stl"/>
+        </geometry>
+        <material name="Ensenso/Blue"/>
+      </visual>
+      <collision>
+        <material name="Ensenso/Black"/>
+        <origin rpy="0 0 0" xyz="0 0.00 0.0219"/>
+        <geometry>
+          <box size="${margin+0.130} ${margin+0.045} ${margin+0.0438}"/>
+        </geometry>
+      </collision>
+    </link>
+    <!-- Left lens -->
+    <joint name="${name}_left_lense_joint" type="fixed">
+      <parent link="${name}"/>
+      <child link="${name}_left_lens_frame"/>
+      <origin xyz="-0.045 0.00 0.05" rpy="0 0 0"/>
+    </joint>
+    <link name="${name}_left_lens_frame"/>
+  </xacro:macro>
+  <xacro:macro name="ensenso_N3x_Series" params="name margin:=0.03">
+    <link name="${name}">
+      <visual>
+        <origin rpy="0 0 0" xyz="0.00 0.0 0.0"/>
+        <geometry>
+          <mesh filename="package://ensenso_description/stl_meshes/N3x.stl"/>
         </geometry>
         <material name="Ensenso/Blue"/>
@@ -28,33 +48,38 @@
       </collision>
     </link>
-    <!-- Projector -->
-    <joint name="${camera}_projector_joint" type="fixed">
-      <parent link="${camera}_mounting_frame"/>
-      <child link="${camera}_projector_lens_frame"/>
-      <origin xyz="0 0.00 0.05" rpy=" 0 0 0"/>
+    <!-- Left lens -->
+    <joint name="${name}_left_lense_joint" type="fixed">
+      <parent link="${name}"/>
+      <child link="${name}_left_lens_frame"/>
+      <origin xyz="-0.05 0.00 0.05" rpy="0 0 0"/>
     </joint>
-    <link name="${camera}_projector_lens_frame"/>
+    <link name="${name}_left_lens_frame"/>
+  </xacro:macro>
+  <xacro:macro name="ensenso_N4x_Series" params="name margin:=0.03">
+    <link name="${name}">
+      <visual>
+        <origin rpy="0 0 0" xyz="0.00 0.0 0.0"/>
+        <geometry>
+          <mesh filename="package://ensenso_description/stl_meshes/N4x.stl"/>
+        </geometry>
+        <material name="Ensenso/Blue"/>
+      </visual>
+      <collision>
+        <origin rpy="0 0 0" xyz="-0.0085 0.00 0.026"/>
+        <geometry>
+          <box size="${margin+0.192} ${margin+0.050} ${margin+0.052}"/>
+        </geometry>
+      </collision>
+    </link>
     <!-- Left lens -->
-    <joint name="${camera}_left_lense_joint" type="fixed">
-      <parent link="${camera}_mounting_frame"/>
-      <child link="${camera}_left_lens_frame"/>
-      <origin xyz="-0.05 0.00 0.05" rpy=" 0 0 0"/>
+    <joint name="${name}_left_lense_joint" type="fixed">
+      <parent link="${name}"/>
+      <child link="${name}_left_lens_frame"/>
+      <origin xyz="-0.05 0.00 0.05" rpy="0 0 0"/>
     </joint>
-    <link name="${camera}_left_lens_frame"/>
-    <!-- Right lens -->
-    <joint name="${camera}_right_lens_joint" type="fixed">
-      <parent link="${camera}_mounting_frame"/>
-      <child link="${camera}_right_lens_frame"/>
-      <origin xyz="0.05 0.00 0.05" rpy=" 0 0 0"/>
-    </joint>
-    <link name="${camera}_right_lens_frame"/>
+    <link name="${name}_left_lens_frame"/>
   </xacro:macro>
-  <xacro:macro name="ensenso_X200_Series" params="camera parent *origin margin radius_lens_sensor length_lens_sensor radius_lens_projector length_lens_projector">
-    <joint name="${parent}_${camera}_joint" type="fixed">
-      <xacro:insert_block name="origin"/>
-      <parent link="${parent}" />
-      <child link="${camera}_mounting_frame" />
-    </joint>
-    <link name="${camera}_mounting_frame">
+  <xacro:macro name="ensenso_X200_Series" params="name margin:=0.03">
+    <link name="${name}">
       <visual>
         <origin rpy="0 0 0" xyz="0 0 0"/>
@@ -65,39 +90,44 @@
       </visual>
       <collision>
-        <origin rpy="0.0 0.0 0.0" xyz="0.0 0.0005 0.033"/>
+        <origin rpy="0.0 0.0 0.0" xyz="0.0 0.0 ${0.033+0.05/2}"/>
         <geometry>
-          <box size="${margin+0.24350} ${margin+0.08} ${margin+0.066}"/>
+          <box size="${margin+0.24350} ${margin+0.066} ${margin+0.08+0.05}"/>
         </geometry>
       </collision>
     </link>
     <!-- Left lens -->
-    <joint name="${camera}_left_lens_joint" type="fixed">
-      <parent link="${camera}_mounting_frame"/>
-      <child link="${camera}_left_lens_frame"/>
-      <origin xyz="-0.1067 0.036 0.033" rpy="-1.570796 0 0"/>
+    <joint name="${name}_left_lens_joint" type="fixed">
+      <parent link="${name}"/>
+      <child link="${name}_left_lens_frame"/>
+      <origin xyz="-0.1067 0.0 0.063" rpy="0 0 0"/>
     </joint>
-    <xacro:objective camera="${camera}" margin="${margin}" name="left" radius="${radius_lens_sensor}" length_tube="${length_lens_sensor}"/>
-    <!-- Right lens -->
-    <joint name="${camera}_right_lens_joint" type="fixed">
-      <parent link="${camera}_mounting_frame"/>
-      <child link="${camera}_right_lens_frame"/>
-      <origin xyz="0.1067 0.036 0.033" rpy="-1.570796 0 0"/>
+    <link name="${name}_left_lens_frame"/>
+  </xacro:macro>
+  <xacro:macro name="ensenso_X200_xFA_Series" params="name margin:=0.03 radius_lens_sensor:=0.02 length_lens_sensor:=0.05">
+    <link name="${name}">
+      <visual>
+        <origin rpy="0 0 0" xyz="0 0 0"/>
+        <geometry>
+          <mesh filename="package://ensenso_description/stl_meshes/X3x-xFA-200.stl"/>
+        </geometry>
+        <material name="Ensenso/Blue"/>
+      </visual>
+      <collision>
+        <origin rpy="0.0 0.0 0.0" xyz="0.0 0.0 ${0.033+0.05/2}"/>
+        <geometry>
+          <box size="${margin+0.2870} ${margin+0.066} ${margin+0.09+0.05}"/>
+        </geometry>
+      </collision>
+    </link>
+    <!-- Left lens -->
+    <joint name="${name}_left_lens_joint" type="fixed">
+      <parent link="${name}"/>
+      <child link="${name}_left_lens_frame"/>
+      <origin xyz="-0.117 0.0 0.063" rpy="0 0 0"/>
     </joint>
-    <xacro:objective camera="${camera}" margin="${margin}" name="right" radius="${radius_lens_sensor}" length_tube="${length_lens_sensor}"/>
-    <!-- Projector lens -->
-    <joint name="${camera}_projector_lens_joint" type="fixed">
-      <parent link="${camera}_mounting_frame"/>
-      <child link="${camera}_projector_lens_frame"/>
-      <origin xyz="0 0.04 0.033" rpy="-1.570796 0 0"/>
-    </joint>
-    <xacro:objective camera="${camera}" margin="${margin}" name="projector" radius="${radius_lens_projector}" length_tube="${length_lens_projector}"/>
+    <link name="${name}_left_lens_frame"/>
   </xacro:macro>
-  <xacro:macro name="ensenso_X400_Series" params="camera parent *origin margin radius_lens_sensor length_lens_sensor radius_lens_projector length_lens_projector">
-    <joint name="${parent}_${camera}_joint" type="fixed">
-      <xacro:insert_block name="origin"/>
-      <parent link="${parent}" />
-      <child link="${camera}_mounting_frame" />
-    </joint>
-    <link name="${camera}_mounting_frame">
+  <xacro:macro name="ensenso_X400_Series" params="name margin:=0.03">
+    <link name="${name}">
       <visual>
         <origin rpy="0 0 0" xyz="0 0 0"/>
@@ -108,82 +138,20 @@
       </visual>
       <collision>
-        <origin rpy="0.0 0.0 0.0" xyz="0.0 0.0005 0.033"/>
+        <origin rpy="0.0 0.0 0.0" xyz="0.0 0.0 ${0.033+0.05/2}"/>
         <geometry>
-          <box size="${margin+0.4515} ${margin+0.08} ${margin+0.066}"/>
+          <box size="${margin+0.4515} ${margin+0.066} ${margin+0.08+0.05}"/>
         </geometry>
       </collision>
     </link>
     <!-- Left lens -->
-    <joint name="${camera}_left_lens_joint" type="fixed">
-      <parent link="${camera}_mounting_frame"/>
-      <child link="${camera}_left_lens_frame"/>
-      <origin xyz="-0.2109 0.036 0.033" rpy="-1.570796 0 0"/>
+    <joint name="${name}_left_lens_joint" type="fixed">
+      <parent link="${name}"/>
+      <child link="${name}_left_lens_frame"/>
+      <origin xyz="-0.2109 0.0 0.063" rpy="0 0 0"/>
     </joint>
-    <xacro:objective camera="${camera}" margin="${margin}" name="left" radius="${radius_lens_sensor}" length_tube="${length_lens_sensor}"/>
-    <!-- Right lens -->
-    <joint name="${camera}_right_lens_joint" type="fixed">
-      <parent link="${camera}_mounting_frame"/>
-      <child link="${camera}_right_lens_frame"/>
-      <origin xyz="0.2109 0.036 0.033" rpy="-1.570796 0 0"/>
-    </joint>
-    <xacro:objective camera="${camera}" margin="${margin}" name="right" radius="${radius_lens_sensor}" length_tube="${length_lens_sensor}"/>
-    <!-- Projector lens -->
-    <joint name="${camera}_projector_lens_joint" type="fixed">
-      <parent link="${camera}_mounting_frame"/>
-      <child link="${camera}_projector_lens_frame"/>
-      <origin xyz="0 0.04 0.033" rpy="-1.570796 0 0"/>
-    </joint>
-    <xacro:objective camera="${camera}" margin="${margin}" name="projector" radius="${radius_lens_projector}" length_tube="${length_lens_projector}"/>
+    <link name="${name}_left_lens_frame"/>
   </xacro:macro>
-  <xacro:macro name="ensenso_X200_xFA_Series" params="camera parent *origin margin radius_lens_sensor length_lens_sensor radius_lens_projector length_lens_projector">
-    <joint name="${parent}_${camera}_joint" type="fixed">
-      <xacro:insert_block name="origin"/>
-      <parent link="${parent}" />
-      <child link="${camera}_mounting_frame" />
-    </joint>
-    <link name="${camera}_mounting_frame">
-      <visual>
-        <origin rpy="0 0 0" xyz="0 0 0"/>
-        <geometry>
-          <mesh filename="package://ensenso_description/stl_meshes/X3x-xFA-200.stl"/>
-        </geometry>
-        <material name="Ensenso/Blue"/>
-      </visual>
-      <collision>
-        <origin rpy="0.0 0.0 0.0" xyz="0.0 -0.004 0.033"/>
-        <geometry>
-          <box size="${margin+0.2870} ${margin+0.09} ${margin+0.066}"/>
-        </geometry>
-      </collision>
-    </link>
-    <!-- Left lens -->
-    <joint name="${camera}_left_lens_joint" type="fixed">
-      <parent link="${camera}_mounting_frame"/>
-      <child link="${camera}_left_lens_frame"/>
-      <origin xyz="-0.117 0.031 0.033" rpy="-1.570796 0 0"/>
-    </joint>
-    <xacro:objective camera="${camera}" margin="${margin}" name="left" radius="${radius_lens_sensor}" length_tube="${length_lens_sensor}"/>
-    <!-- Right lens -->
-    <joint name="${camera}_right_lens_joint" type="fixed">
-      <parent link="${camera}_mounting_frame"/>
-      <child link="${camera}_right_lens_frame"/>
-      <origin xyz="0.117 0.031 0.033" rpy="-1.570796 0 0"/>
-    </joint>
-    <xacro:objective camera="${camera}" margin="${margin}" name="right" radius="${radius_lens_sensor}" length_tube="${length_lens_sensor}"/>
-    <!-- Projector lens -->
-    <joint name="${camera}_projector_lens_joint" type="fixed">
-      <parent link="${camera}_mounting_frame"/>
-      <child link="${camera}_projector_lens_frame"/>
-      <origin xyz="0 0.041 0.033" rpy="-1.570796 0 0"/>
-    </joint>
-    <xacro:objective camera="${camera}" margin="${margin}" name="projector" radius="${radius_lens_projector}" length_tube="${length_lens_projector}"/>
-  </xacro:macro>
-  <xacro:macro name="ensenso_X400_xFA_Series" params="camera parent *origin margin radius_lens_sensor length_lens_sensor radius_lens_projector length_lens_projector">
-    <joint name="${parent}_${camera}_joint" type="fixed">
-      <xacro:insert_block name="origin"/>
-      <parent link="${parent}" />
-      <child link="${camera}_mounting_frame" />
-    </joint>
-    <link name="${camera}_mounting_frame">
+  <xacro:macro name="ensenso_X400_xFA_Series" params="name margin:=0.03">
+    <link name="${name}">
       <visual>
         <origin rpy="0 0 0" xyz="0 0 0"/>
@@ -194,48 +162,17 @@
       </visual>
       <collision>
-        <origin rpy="0.0 0.0 0.0" xyz="0.0 -0.004 0.033"/>
+        <origin rpy="0.0 0.0 0.0" xyz="0.0 0.0 ${0.033+0.05/2}"/>
         <geometry>
-          <box size="${margin+0.4950} ${margin+0.09} ${margin+0.066}"/>
+          <box size="${margin+0.4950} ${margin+0.066} ${margin+0.09+0.05}"/>
         </geometry>
       </collision>
     </link>
     <!-- Left lens -->
-    <joint name="${camera}_left_lens_joint" type="fixed">
-      <parent link="${camera}_mounting_frame"/>
-      <child link="${camera}_left_lens_frame"/>
-      <origin xyz="-0.22125 0.031 0.033" rpy="-1.570796 0 0"/>
+    <joint name="${name}_left_lens_joint" type="fixed">
+      <parent link="${name}"/>
+      <child link="${name}_left_lens_frame"/>
+      <origin xyz="-0.22125 0 0.063" rpy="0 0 0"/>
     </joint>
-    <xacro:objective camera="${camera}" margin="${margin}" name="left" radius="${radius_lens_sensor}" length_tube="${length_lens_sensor}"/>
-    <!-- Right lens -->
-    <joint name="${camera}_right_lens_joint" type="fixed">
-      <parent link="${camera}_mounting_frame"/>
-      <child link="${camera}_right_lens_frame"/>
-      <origin xyz="0.22125 0.031 0.033" rpy="-1.570796 0 0"/>
-    </joint>
-    <xacro:objective camera="${camera}" margin="${margin}" name="right" radius="${radius_lens_sensor}" length_tube="${length_lens_sensor}"/>
-    <!-- Projector lens -->
-    <joint name="${camera}_projector_lens_joint" type="fixed">
-      <parent link="${camera}_mounting_frame"/>
-      <child link="${camera}_projector_lens_frame"/>
-      <origin xyz="0 0.041 0.033" rpy="-1.570796 0 0"/>
-    </joint>
-    <xacro:objective camera="${camera}" margin="${margin}" name="projector" radius="${radius_lens_projector}" length_tube="${length_lens_projector}"/>
-  </xacro:macro>
-  <xacro:macro name="objective" params="camera margin name radius length_tube">
-    <link name="${camera}_${name}_lens_frame">
-      <visual>
-        <origin xyz="0.0 0.0 ${length_tube / 2.0}" rpy="0 0 0"/>
-        <geometry>
-          <cylinder length="${length_tube}" radius="${radius}"/>
-        </geometry>
-        <material name="Ensenso/Black"/>
-      </visual>
-      <collision>
-        <origin xyz="0.0 0.0 ${(length_tube+2*margin) / 2.0}" rpy="0 0 0"/>
-        <geometry>
-          <cylinder length="${length_tube+2*margin}" radius="${radius+margin}"/>
-        </geometry>
-      </collision>
-    </link>
+    <link name="${name}_left_lens_frame"/>
   </xacro:macro>
 </robot>
