Commit message: add N4x / refactor examples

File: ensenso_description/ensenso.xacro (robot description, xacro)
@@ -7,5 +7,5 @@
   <color rgba="0.0 0.0 0.0 1.0"/>
 </material>
-  <xacro:macro name="ensenso_N_Series" params="name margin:=0.03">
+  <xacro:macro name="ensenso_N3x_Series" params="name margin:=0.03">
     <link name="${name}">
       <visual>
@@ -45,4 +45,42 @@
     <link name="${name}_right_lens_frame"/>
   </xacro:macro>
+  <xacro:macro name="ensenso_N4x_Series" params="name margin:=0.03">
+    <link name="${name}">
+      <visual>
+        <origin rpy="0 0 0" xyz="0.00 0.0 0.0"/>
+        <geometry>
+          <mesh filename="package://ensenso_description/stl_meshes/N4x-xxx.stl"/>
+        </geometry>
+        <material name="Ensenso/Blue"/>
+      </visual>
+      <collision>
+        <origin rpy="0 0 0" xyz="-0.0085 0.00 0.026"/>
+        <geometry>
+          <box size="${margin+0.192} ${margin+0.050} ${margin+0.052}"/>
+        </geometry>
+      </collision>
+    </link>
+    <!-- Projector -->
+    <joint name="${name}_projector_joint" type="fixed">
+      <parent link="${name}"/>
+      <child link="${name}_projector_lens_frame"/>
+      <origin xyz="0 0.00 0.05" rpy=" 0 0 0"/>
+    </joint>
+    <link name="${name}_projector_lens_frame"/>
+    <!-- Left lens -->
+    <joint name="${name}_left_lense_joint" type="fixed">
+      <parent link="${name}"/>
+      <child link="${name}_left_lens_frame"/>
+      <origin xyz="-0.05 0.00 0.05" rpy=" 0 0 0"/>
+    </joint>
+    <link name="${name}_left_lens_frame"/>
+    <!-- Right lens -->
+    <joint name="${name}_right_lens_joint" type="fixed">
+      <parent link="${name}"/>
+      <child link="${name}_right_lens_frame"/>
+      <origin xyz="0.05 0.00 0.05" rpy=" 0 0 0"/>
+    </joint>
+    <link name="${name}_right_lens_frame"/>
+  </xacro:macro>
   <xacro:macro name="ensenso_X200_Series" params="name margin:=0.03 radius_lens_sensor:=0.02 length_lens_sensor:=0.05 radius_lens_projector:=0.02 length_lens_projector:=0.05">
     <link name="${name}">

File: ensenso_description/ensenso_N3x_Series.xacro (robot description, xacro)
@@ -2,6 +2,6 @@
 <robot name="ensenso_camera" xmlns:xacro="http://www.ros.org/wiki/xacro">
   <xacro:include filename="$(find ensenso_description)/ensenso.xacro" />
-  <xacro:property name="camera_name" default="X200_xFA" />
-  <xacro:ensenso_X400_Series name="${camera_name}" />
+  <xacro:property name="camera_name" default="N35" />
+  <xacro:ensenso_N3x_Series name="${camera_name}" />
   <joint name="world_to_${camera_name}" type="fixed">
     <parent link="base_link" />
@@ -12,4 +12,4 @@
 </robot>
 <!-- example usage with:
-  roslaunch urdf_tutorial display.launch model:=`rospack find ensenso_description`/ensenso_X400_Series.xacro gui:=true
+  roslaunch urdf_tutorial display.launch model:=`rospack find ensenso_description`/ensenso_N3x_Series.xacro gui:=true
 -->

File: ensenso_description/ensenso_N4x_Series.xacro (robot description, xacro)
@@ -2,6 +2,6 @@
 <robot name="ensenso_camera" xmlns:xacro="http://www.ros.org/wiki/xacro">
   <xacro:include filename="$(find ensenso_description)/ensenso.xacro" />
-  <xacro:property name="camera_name" default="X200_xFA" />
-  <xacro:ensenso_X400_Series name="${camera_name}" />
+  <xacro:property name="camera_name" default="N35" />
+  <xacro:ensenso_N4x_Series name="${camera_name}" />
   <joint name="world_to_${camera_name}" type="fixed">
     <parent link="base_link" />
@@ -12,4 +12,4 @@
 </robot>
 <!-- example usage with:
-  roslaunch urdf_tutorial display.launch model:=`rospack find ensenso_description`/ensenso_X400_Series.xacro gui:=true
+  roslaunch urdf_tutorial display.launch model:=`rospack find ensenso_description`/ensenso_N4x_Series.xacro gui:=true
 -->

File: ensenso_description/ensenso_X200_Series.xacro (robot description, xacro)
@@ -2,28 +2,13 @@
 <robot name="ensenso_camera" xmlns:xacro="http://www.ros.org/wiki/xacro">
   <xacro:include filename="$(find ensenso_description)/ensenso.xacro" />
-  <!-- Parameters -->
-  <!-- Name of the camera -->
-  <xacro:arg name="camera" default="X200" />
-  <xacro:property name="camera" value="$(arg camera)" />
-  <!-- Enlarges the bounding box in all directions -->
-  <xacro:arg name="margin" default="0.03" />
-  <xacro:property name="margin" value="$(arg margin)" />
-  <!-- Lens objective properties -->
-  <xacro:arg name="lens_length" default="0.05" />
-  <xacro:property name="lens_length" value="$(arg lens_length)"/>
-  <xacro:arg name="lens_radius" default="0.02" />
-  <xacro:property name="lens_radius" value="$(arg lens_radius)"/>
-  <!-- Projector objective properties -->
-  <xacro:arg name="projector_length" default="0.05" />
-  <xacro:property name="projector_length" value="$(arg projector_length)" />
-  <xacro:arg name="projector_radius" default="0.02" />
-  <xacro:property name="projector_radius" value="$(arg projector_radius)" />
-  <!-- Tf Frame, that references to the cameras mounting frame -->
-  <xacro:arg name="corresponding_frame_name" default="world" />
-  <xacro:property name="corresponding_frame_name" value="$(arg corresponding_frame_name)" />
-  <link name="${corresponding_frame_name}"/>
-  <xacro:ensenso_X200_Series camera="${camera}" parent="${corresponding_frame_name}" margin="${margin}" radius_lens_sensor="${lens_radius}" length_lens_sensor="${lens_length}" radius_lens_projector="${projector_radius}" length_lens_projector="${projector_length}">
-    <origin xyz="0 0 0.0" rpy="0 0 0" />
-  </xacro:ensenso_X200_Series>
-</robot>
-<!-- example usage with: roslaunch urdf_tutorial display.launch model:=`rospack find ensenso_description`/ensenso_X200_Series.xacro gui:=true -->
+  <xacro:property name="camera_name" default="X200" />
+  <xacro:ensenso_X200_Series name="${camera_name}" />
+  <joint name="world_to_${camera_name}" type="fixed">
+    <parent link="base_link" />
+    <child link="${camera_name}" />
+    <origin xyz="0 0 0" rpy="0 0 0" />
+  </joint>
+  <link name="base_link" />
+</robot><!-- example usage with:
+  roslaunch urdf_tutorial display.launch model:=`rospack find ensenso_description`/ensenso_X200_Series.xacro gui:=true
+-->

File: ensenso_description/ensenso_X200_xFA_Series.xacro (robot description, xacro)
@@ -2,28 +2,14 @@
 <robot name="ensenso_camera" xmlns:xacro="http://www.ros.org/wiki/xacro">
   <xacro:include filename="$(find ensenso_description)/ensenso.xacro" />
-  <!-- Parameters -->
-  <!-- Name of the camera -->
-  <xacro:arg name="camera" default="X200_xFA" />
-  <xacro:property name="camera" value="$(arg camera)" />
-  <!-- Enlarges the bounding box in all directions -->
-  <xacro:arg name="margin" default="0.03" />
-  <xacro:property name="margin" value="$(arg margin)" />
-  <!-- Lens objective properties -->
-  <xacro:arg name="lens_length" default="0.05" />
-  <xacro:property name="lens_length" value="$(arg lens_length)"/>
-  <xacro:arg name="lens_radius" default="0.02" />
-  <xacro:property name="lens_radius" value="$(arg lens_radius)"/>
-  <!-- Projector objective properties -->
-  <xacro:arg name="projector_length" default="0.05" />
-  <xacro:property name="projector_length" value="$(arg projector_length)" />
-  <xacro:arg name="projector_radius" default="0.02" />
-  <xacro:property name="projector_radius" value="$(arg projector_radius)" />
-  <!-- Tf Frame, that references to the cameras mounting frame -->
-  <xacro:arg name="corresponding_frame_name" default="world" />
-  <xacro:property name="corresponding_frame_name" value="$(arg corresponding_frame_name)" />
-  <link name="${corresponding_frame_name}"/>
-  <xacro:ensenso_X200_xFA_Series camera="${camera}" parent="${corresponding_frame_name}" margin="${margin}" radius_lens_sensor="${lens_radius}" length_lens_sensor="${lens_length}" radius_lens_projector="${projector_radius}" length_lens_projector="${projector_length}">
-    <origin xyz="0 0 0.0" rpy="0 0 0" />
-  </xacro:ensenso_X200_xFA_Series>
+  <xacro:property name="camera_name" default="X200_xFA" />
+  <xacro:ensenso_X200_xFA_Series name="${camera_name}" />
+  <joint name="world_to_${camera_name}" type="fixed">
+    <parent link="base_link" />
+    <child link="${camera_name}" />
+    <origin xyz="0 0 0" rpy="0 0 0" />
+  </joint>
+  <link name="base_link" />
 </robot>
-<!-- example usage with: roslaunch urdf_tutorial display.launch model:=`rospack find ensenso_description`/ensenso_X200_xFA_Series.xacro gui:=true -->
+<!-- example usage with:
+  roslaunch urdf_tutorial display.launch model:=`rospack find ensenso_description`/ensenso_X200_xFA_Series.xacro gui:=true
+-->

File: ensenso_description/ensenso_X400_xFA_Series.xacro (robot description, xacro)
@@ -2,28 +2,14 @@
 <robot name="ensenso_camera" xmlns:xacro="http://www.ros.org/wiki/xacro">
   <xacro:include filename="$(find ensenso_description)/ensenso.xacro" />
-  <!-- Parameters -->
-  <!-- Name of the camera -->
-  <xacro:arg name="camera" default="X400_xFA" />
-  <xacro:property name="camera" value="$(arg camera)" />
-  <!-- Enlarges the bounding box in all directions -->
-  <xacro:arg name="margin" default="0.03" />
-  <xacro:property name="margin" value="$(arg margin)" />
-  <!-- Lens objective properties -->
-  <xacro:arg name="lens_length" default="0.05" />
-  <xacro:property name="lens_length" value="$(arg lens_length)"/>
-  <xacro:arg name="lens_radius" default="0.02" />
-  <xacro:property name="lens_radius" value="$(arg lens_radius)"/>
-  <!-- Projector objective properties -->
-  <xacro:arg name="projector_length" default="0.05" />
-  <xacro:property name="projector_length" value="$(arg projector_length)" />
-  <xacro:arg name="projector_radius" default="0.02" />
-  <xacro:property name="projector_radius" value="$(arg projector_radius)" />
-  <!-- Tf Frame, that references to the cameras mounting frame -->
-  <xacro:arg name="corresponding_frame_name" default="world" />
-  <xacro:property name="corresponding_frame_name" value="$(arg corresponding_frame_name)" />
-  <link name="${corresponding_frame_name}"/>
-  <xacro:ensenso_X400_xFA_Series camera="${camera}" parent="${corresponding_frame_name}" margin="${margin}" radius_lens_sensor="${lens_radius}" length_lens_sensor="${lens_length}" radius_lens_projector="${projector_radius}" length_lens_projector="${projector_length}">
-    <origin xyz="0 0 0.0" rpy="0 0 0" />
-  </xacro:ensenso_X400_xFA_Series>
+  <xacro:property name="camera_name" default="X200_xFA" />
+  <xacro:ensenso_X400_xFA_Series name="${camera_name}" />
+  <joint name="world_to_${camera_name}" type="fixed">
+    <parent link="base_link" />
+    <child link="${camera_name}" />
+    <origin xyz="0 0 0" rpy="0 0 0" />
+  </joint>
+  <link name="base_link" />
 </robot>
-<!-- example usage with: roslaunch urdf_tutorial display.launch model:=`rospack find ensenso_description`/ensenso_X400_xFA_Series.xacro gui:=true -->
+<!-- example usage with:
+  roslaunch urdf_tutorial display.launch model:=`rospack find ensenso_description`/ensenso_X400_xFA_Series.xacro gui:=true
+-->
