Commit message: remove projector- and right_lens-links & projector-objective == sensor-objective

File: ensenso_description/ensenso.xacro (robot description, xacro)
@@ -23,11 +23,4 @@
       </collision>
     </link>
-    <!-- Projector -->
-    <joint name="${name}_projector_joint" type="fixed">
-      <parent link="${name}"/>
-      <child link="${name}_projector_lens_frame"/>
-      <origin xyz="0 0.00 0.05" rpy=" 0 0 0"/>
-    </joint>
-    <link name="${name}_projector_lens_frame"/>
     <!-- Left lens -->
     <joint name="${name}_left_lense_joint" type="fixed">
@@ -37,11 +30,4 @@
     </joint>
     <link name="${name}_left_lens_frame"/>
-    <!-- Right lens -->
-    <joint name="${name}_right_lens_joint" type="fixed">
-      <parent link="${name}"/>
-      <child link="${name}_right_lens_frame"/>
-      <origin xyz="0.05 0.00 0.05" rpy=" 0 0 0"/>
-    </joint>
-    <link name="${name}_right_lens_frame"/>
   </xacro:macro>
   <xacro:macro name="ensenso_N4x_Series" params="name margin:=0.03">
@@ -61,11 +47,4 @@
       </collision>
     </link>
-    <!-- Projector -->
-    <joint name="${name}_projector_joint" type="fixed">
-      <parent link="${name}"/>
-      <child link="${name}_projector_lens_frame"/>
-      <origin xyz="0 0.00 0.05" rpy=" 0 0 0"/>
-    </joint>
-    <link name="${name}_projector_lens_frame"/>
     <!-- Left lens -->
     <joint name="${name}_left_lense_joint" type="fixed">
@@ -75,13 +54,6 @@
     </joint>
     <link name="${name}_left_lens_frame"/>
-    <!-- Right lens -->
-    <joint name="${name}_right_lens_joint" type="fixed">
-      <parent link="${name}"/>
-      <child link="${name}_right_lens_frame"/>
-      <origin xyz="0.05 0.00 0.05" rpy=" 0 0 0"/>
-    </joint>
-    <link name="${name}_right_lens_frame"/>
-  </xacro:macro>
-  <xacro:macro name="ensenso_X200_Series" params="name margin:=0.03 radius_lens_sensor:=0.02 length_lens_sensor:=0.05 radius_lens_projector:=0.02 length_lens_projector:=0.05">
+  </xacro:macro>
+  <xacro:macro name="ensenso_X200_Series" params="name margin:=0.03 radius_lens_sensor:=0.02 length_lens_sensor:=0.05">
     <link name="${name}">
       <visual>
@@ -92,8 +64,17 @@
         <material name="Ensenso/Blue"/>
       </visual>
-      <collision>
-        <origin rpy="0.0 0.0 0.0" xyz="0.0 0.0005 0.033"/>
-        <geometry>
-          <box size="${margin+0.24350} ${margin+0.08} ${margin+0.066}"/>
+      <xacro:objective radius="${radius_lens_sensor}" length_tube="${length_lens_sensor}">
+        <origin xyz="-0.1067 ${0.036+length_lens_sensor/2.0} 0.033" rpy="${-pi/2} 0 0"/>
+      </xacro:objective>
+      <xacro:objective radius="${radius_lens_sensor}" length_tube="${length_lens_sensor}">
+        <origin xyz="0.1067 ${0.036+length_lens_sensor/2.0} 0.033" rpy="-1.570796 0 0"/>
+      </xacro:objective>
+      <xacro:objective radius="${radius_lens_sensor}" length_tube="${length_lens_sensor}">
+        <origin xyz="0 ${0.04+length_lens_sensor/2.0} 0.033" rpy="-1.570796 0 0"/>
+      </xacro:objective>
+      <collision>
+        <origin rpy="0.0 0.0 0.0" xyz="0.0 ${0.0005+length_lens_sensor/2} 0.033"/>
+        <geometry>
+          <box size="${margin+0.24350} ${margin+0.08+length_lens_sensor} ${margin+0.066}"/>
         </geometry>
       </collision>
@@ -105,21 +86,40 @@
       <origin xyz="-0.1067 0.036 0.033" rpy="-1.570796 0 0"/>
     </joint>
-    <xacro:objective name="${name}" margin="${margin}" identifier="left" radius="${radius_lens_sensor}" length_tube="${length_lens_sensor}"/>
-    <!-- Right lens -->
-    <joint name="${name}_right_lens_joint" type="fixed">
-      <parent link="${name}"/>
-      <child link="${name}_right_lens_frame"/>
-      <origin xyz="0.1067 0.036 0.033" rpy="-1.570796 0 0"/>
-    </joint>
-    <xacro:objective name="${name}" margin="${margin}" identifier="right" radius="${radius_lens_sensor}" length_tube="${length_lens_sensor}"/>
-    <!-- Projector lens -->
-    <joint name="${name}_projector_lens_joint" type="fixed">
-      <parent link="${name}"/>
-      <child link="${name}_projector_lens_frame"/>
-      <origin xyz="0 0.04 0.033" rpy="-1.570796 0 0"/>
-    </joint>
-    <xacro:objective name="${name}" margin="${margin}" identifier="projector" radius="${radius_lens_projector}" length_tube="${length_lens_projector}"/>
-  </xacro:macro>
-  <xacro:macro name="ensenso_X400_Series" params="name margin:=0.03 radius_lens_sensor:=0.02 length_lens_sensor:=0.05 radius_lens_projector:=0.02 length_lens_projector:=0.05">
+    <link name="${name}_left_lens_frame"/>
+  </xacro:macro>
+  <xacro:macro name="ensenso_X200_xFA_Series" params="name margin:=0.03 radius_lens_sensor:=0.02 length_lens_sensor:=0.05">
+    <link name="${name}">
+      <visual>
+        <origin rpy="0 0 0" xyz="0 0 0"/>
+        <geometry>
+          <mesh filename="package://ensenso_description/stl_meshes/X3x-xFA-200.stl"/>
+        </geometry>
+        <material name="Ensenso/Blue"/>
+      </visual>
+      <xacro:objective radius="${radius_lens_sensor}" length_tube="${length_lens_sensor}">
+        <origin xyz="-0.117 ${0.031+length_lens_sensor/2.0} 0.033" rpy="${-pi/2} 0 0"/>
+      </xacro:objective>
+      <xacro:objective radius="${radius_lens_sensor}" length_tube="${length_lens_sensor}">
+        <origin xyz="0.117 ${0.031+length_lens_sensor/2.0} 0.033" rpy="-1.570796 0 0"/>
+      </xacro:objective>
+      <xacro:objective radius="${radius_lens_sensor}" length_tube="${length_lens_sensor}">
+        <origin xyz="0 ${0.041+length_lens_sensor/2.0} 0.033" rpy="-1.570796 0 0"/>
+      </xacro:objective>
+      <collision>
+        <origin rpy="0.0 0.0 0.0" xyz="0.0 ${-0.004+length_lens_sensor/2} 0.033"/>
+        <geometry>
+          <box size="${margin+0.2870} ${margin+0.09+length_lens_sensor} ${margin+0.066}"/>
+        </geometry>
+      </collision>
+    </link>
+    <!-- Left lens -->
+    <joint name="${name}_left_lens_joint" type="fixed">
+      <parent link="${name}"/>
+      <child link="${name}_left_lens_frame"/>
+      <origin xyz="-0.117 0.031 0.033" rpy="-1.570796 0 0"/>
+    </joint>
+    <link name="${name}_left_lens_frame"/>
+  </xacro:macro>
+  <xacro:macro name="ensenso_X400_Series" params="name margin:=0.03 radius_lens_sensor:=0.02 length_lens_sensor:=0.05">
     <link name="${name}">
       <visual>
@@ -130,8 +130,17 @@
         <material name="Ensenso/Blue"/>
       </visual>
-      <collision>
-        <origin rpy="0.0 0.0 0.0" xyz="0.0 0.0005 0.033"/>
-        <geometry>
-          <box size="${margin+0.4515} ${margin+0.08} ${margin+0.066}"/>
+      <xacro:objective radius="${radius_lens_sensor}" length_tube="${length_lens_sensor}">
+        <origin xyz="-0.2109 ${0.036+length_lens_sensor/2.0} 0.033" rpy="${-pi/2} 0 0"/>
+      </xacro:objective>
+      <xacro:objective radius="${radius_lens_sensor}" length_tube="${length_lens_sensor}">
+        <origin xyz="0.2109 ${0.036+length_lens_sensor/2.0} 0.033" rpy="-1.570796 0 0"/>
+      </xacro:objective>
+      <xacro:objective radius="${radius_lens_sensor}" length_tube="${length_lens_sensor}">
+        <origin xyz="0 ${0.04+length_lens_sensor/2.0} 0.033" rpy="-1.570796 0 0"/>
+      </xacro:objective>
+      <collision>
+        <origin rpy="0.0 0.0 0.0" xyz="0.0 ${0.0005+length_lens_sensor/2} 0.033"/>
+        <geometry>
+          <box size="${margin+0.4515} ${margin+0.08+length_lens_sensor} ${margin+0.066}"/>
         </geometry>
       </collision>
@@ -143,70 +152,33 @@
       <origin xyz="-0.2109 0.036 0.033" rpy="-1.570796 0 0"/>
     </joint>
-    <xacro:objective name="${name}" margin="${margin}" identifier="left" radius="${radius_lens_sensor}" length_tube="${length_lens_sensor}"/>
-    <!-- Right lens -->
-    <joint name="${name}_right_lens_joint" type="fixed">
-      <parent link="${name}"/>
-      <child link="${name}_right_lens_frame"/>
-      <origin xyz="0.2109 0.036 0.033" rpy="-1.570796 0 0"/>
-    </joint>
-    <xacro:objective name="${name}" margin="${margin}" identifier="right" radius="${radius_lens_sensor}" length_tube="${length_lens_sensor}"/>
-    <!-- Projector lens -->
-    <joint name="${name}_projector_lens_joint" type="fixed">
-      <parent link="${name}"/>
-      <child link="${name}_projector_lens_frame"/>
-      <origin xyz="0 0.04 0.033" rpy="-1.570796 0 0"/>
-    </joint>
-    <xacro:objective name="${name}" margin="${margin}" identifier="projector" radius="${radius_lens_projector}" length_tube="${length_lens_projector}"/>
-  </xacro:macro>
-  <xacro:macro name="ensenso_X200_xFA_Series" params="name margin:=0.03 radius_lens_sensor:=0.02 length_lens_sensor:=0.05 radius_lens_projector:=0.02 length_lens_projector:=0.05">
-    <link name="${name}">
-      <visual>
-        <origin rpy="0 0 0" xyz="0 0 0"/>
-        <geometry>
-          <mesh filename="package://ensenso_description/stl_meshes/X3x-xFA-200.stl"/>
-        </geometry>
-        <material name="Ensenso/Blue"/>
-      </visual>
+    <link name="${name}_left_lens_frame"/>
+  </xacro:macro>
+  <xacro:macro name="ensenso_X400_xFA_Series" params="name margin:=0.03 radius_lens_sensor:=0.02 length_lens_sensor:=0.05 radius_lens_projector:=0.02 length_lens_projector:=0.05">
+    <link name="${name}">
+      <visual>
+        <origin rpy="0 0 0" xyz="0 0 0"/>
+        <geometry>
+          <mesh filename="package://ensenso_description/stl_meshes/X3x-xFA-400.stl"/>
+        </geometry>
+        <material name="Ensenso/Blue"/>
+      </visual>
+      <xacro:objective radius="${radius_lens_sensor}" length_tube="${length_lens_sensor}">
+        <origin xyz="-0.22125 ${0.031+length_lens_sensor/2.0} 0.033" rpy="${-pi/2} 0 0"/>
+      </xacro:objective>
+      <xacro:objective radius="${radius_lens_sensor}" length_tube="${length_lens_sensor}">
+        <origin xyz="0.22125 ${0.031+length_lens_sensor/2.0} 0.033" rpy="-1.570796 0 0"/>
+      </xacro:objective>
+      <xacro:objective radius="${radius_lens_sensor}" length_tube="${length_lens_sensor}">
+        <origin xyz="0 ${0.041+length_lens_sensor/2.0} 0.033" rpy="-1.570796 0 0"/>
+      </xacro:objective>
+      <collision>
+        <origin rpy="0.0 0.0 0.0" xyz="0.0 ${-0.004+length_lens_sensor/2} 0.033"/>
+        <geometry>
+          <box size="${margin+0.4950} ${margin+0.09+length_lens_sensor} ${margin+0.066}"/>
+        </geometry>
+      </collision>
       <collision>
         <origin rpy="0.0 0.0 0.0" xyz="0.0 -0.004 0.033"/>
         <geometry>
-          <box size="${margin+0.2870} ${margin+0.09} ${margin+0.066}"/>
-        </geometry>
-      </collision>
-    </link>
-    <!-- Left lens -->
-    <joint name="${name}_left_lens_joint" type="fixed">
-      <parent link="${name}"/>
-      <child link="${name}_left_lens_frame"/>
-      <origin xyz="-0.117 0.031 0.033" rpy="-1.570796 0 0"/>
-    </joint>
-    <xacro:objective name="${name}" margin="${margin}" identifier="left" radius="${radius_lens_sensor}" length_tube="${length_lens_sensor}"/>
-    <!-- Right lens -->
-    <joint name="${name}_right_lens_joint" type="fixed">
-      <parent link="${name}"/>
-      <child link="${name}_right_lens_frame"/>
-      <origin xyz="0.117 0.031 0.033" rpy="-1.570796 0 0"/>
-    </joint>
-    <xacro:objective name="${name}" margin="${margin}" identifier="right" radius="${radius_lens_sensor}" length_tube="${length_lens_sensor}"/>
-    <!-- Projector lens -->
-    <joint name="${name}_projector_lens_joint" type="fixed">
-      <parent link="${name}"/>
-      <child link="${name}_projector_lens_frame"/>
-      <origin xyz="0 0.041 0.033" rpy="-1.570796 0 0"/>
-    </joint>
-    <xacro:objective name="${name}" margin="${margin}" identifier="projector" radius="${radius_lens_projector}" length_tube="${length_lens_projector}"/>
-  </xacro:macro>
-  <xacro:macro name="ensenso_X400_xFA_Series" params="name margin:=0.03 radius_lens_sensor:=0.02 length_lens_sensor:=0.05 radius_lens_projector:=0.02 length_lens_projector:=0.05">
-    <link name="${name}">
-      <visual>
-        <origin rpy="0 0 0" xyz="0 0 0"/>
-        <geometry>
-          <mesh filename="package://ensenso_description/stl_meshes/X3x-xFA-400.stl"/>
-        </geometry>
-        <material name="Ensenso/Blue"/>
-      </visual>
-      <collision>
-        <origin rpy="0.0 0.0 0.0" xyz="0.0 -0.004 0.033"/>
-        <geometry>
           <box size="${margin+0.4950} ${margin+0.09} ${margin+0.066}"/>
         </geometry>
@@ -219,24 +191,9 @@
       <origin xyz="-0.22125 0.031 0.033" rpy="-1.570796 0 0"/>
     </joint>
-    <xacro:objective name="${name}" margin="${margin}" identifier="left" radius="${radius_lens_sensor}" length_tube="${length_lens_sensor}"/>
-    <!-- Right lens -->
-    <joint name="${name}_right_lens_joint" type="fixed">
-      <parent link="${name}"/>
-      <child link="${name}_right_lens_frame"/>
-      <origin xyz="0.22125 0.031 0.033" rpy="-1.570796 0 0"/>
-    </joint>
-    <xacro:objective name="${name}" margin="${margin}" identifier="right" radius="${radius_lens_sensor}" length_tube="${length_lens_sensor}"/>
-    <!-- Projector lens -->
-    <joint name="${name}_projector_lens_joint" type="fixed">
-      <parent link="${name}"/>
-      <child link="${name}_projector_lens_frame"/>
-      <origin xyz="0 0.041 0.033" rpy="-1.570796 0 0"/>
-    </joint>
-    <xacro:objective name="${name}" margin="${margin}" identifier="projector" radius="${radius_lens_projector}" length_tube="${length_lens_projector}"/>
-  </xacro:macro>
-  <xacro:macro name="objective" params="name margin identifier radius length_tube">
-    <link name="${name}_${identifier}_lens_frame">
-      <visual>
-        <origin xyz="0.0 0.0 ${length_tube / 2.0}" rpy="0 0 0"/>
+    <link name="${name}_left_lens_frame"/>
+  </xacro:macro>
+  <xacro:macro name="objective" params="radius length_tube *origin">
+      <visual>
+        <xacro:insert_block name="origin" />
         <geometry>
           <cylinder length="${length_tube}" radius="${radius}"/>
@@ -244,11 +201,4 @@
         <material name="Ensenso/Black"/>
       </visual>
-      <collision>
-        <origin xyz="0.0 0.0 ${(length_tube+2*margin) / 2.0}" rpy="0 0 0"/>
-        <geometry>
-          <cylinder length="${length_tube+2*margin}" radius="${radius+margin}"/>
-        </geometry>
-      </collision>
-    </link>
   </xacro:macro>
 </robot>

Commit message: set correct origin of X3x-FA-200.stl

File: ensenso_description/ensenso.xacro (robot description, xacro)
@@ -104,5 +104,5 @@
     <link name="${name}_left_lens_frame"/>
   </xacro:macro>
-  <xacro:macro name="ensenso_X200_xFA_Series" params="name margin:=0.03 radius_lens_sensor:=0.02 length_lens_sensor:=0.05">
+  <xacro:macro name="ensenso_X200_xFA_Series" params="name margin:=0.03">
     <link name="${name}">
       <visual>
